File: schem1.sch (EAGLE design)
At the start: 0 parts

Commit message: работает без ардуино по кнопкам
Other:
- note added: "CP"
- note added: "D"
- note added: "OE"
- note added: "STR"
Changed lines of the file:
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@@
 <?xml version="1.0" encoding="utf-8"?>
 <!DOCTYPE eagle SYSTEM "eagle.dtd">
-<eagle version="8.6.0">
+<eagle version="8.7.1">
 <drawing>
 <settings>
@@
 <wire x1="124.46" y1="81.28" x2="223.52" y2="81.28" width="0.762" layer="93"/>
 <wire x1="223.52" y1="81.28" x2="223.52" y2="58.42" width="0.762" layer="93"/>
+<text x="1.524" y="54.864" size="3.81" layer="90">OE</text>
+<text x="1.778" y="32.512" size="3.81" layer="90">CP</text>
+<text x="-30.48" y="38.1" size="3.81" layer="90">STR</text>
+<text x="-27.94" y="55.88" size="3.81" layer="90">D</text>
 </plain>
 <moduleinsts>
